Commit message: Fixed errors with simulation

File: ros2_ws/install/robotic_arm_gazebo/share/robotic_arm_gazebo/urdf/robotic_arm.urdf.xacro (robot description, xacro)
@@ -1,5 +1,5 @@
 <?xml version="1.0"?>
 <robot xmlns:xacro="http://www.ros.org/wiki/xacro" name="robotic_arm">
-  <xacro:property name="pi" value="3.14159265359"/>
+  <!-- Note: xacro already provides mathematical constants like pi; avoid redefining to prevent stderr warnings. -->
   <!-- Colors -->
   <material name="gray"><color rgba="0.7 0.7 0.7 1.0"/></material>
